File: AeroSAR_electronics/AeroSAR_electronics.kicad_sch (KiCad schematic)
At the start: 26 parts, among them J1 USB_B_Micro, J10 Servo, J11 Servo, J12 Servo, J13 Servo, J14 NAV Module, J15 RPI, J16 Receiver, J17 PDB, J2 ESC-1, J3 ESC-2, J4 Servo, J5 Servo, J6 Servo, J7 Servo, J8 Servo, J9 Servo, SW1 RESET

Commit message: Added missing connections
Connections:
- net GND-WiFi is gone; now on net GND: C1.2, C2.2
- net GND: now also FC-TOP1.83 (GND), J14.2, J14.A2
