File: AeroSAR_electronics/AeroSAR_electronics.kicad_pcb (KiCad board)
At the start: 2 copper layers, 160 x 80 mm, 26 parts, among them J1 USB_B_Micro, J10 Servo, J11 Servo, J12 Servo, J13 Servo, J14 NAV Module, J15 RPI, J16 Receiver, J17 PDB, J2 ESC-1, J3 ESC-2, J4 Servo, J5 Servo, J6 Servo, J7 Servo, J8 Servo, J9 Servo, SW1 RESET

Commit message: Added missing connections
Parts:
- added G***: LOGO, LOGO, F.Cu at (92.6, 96.2)
- NAV Module: renamed from J14
- renumbered J2 to ESC-1, J3 to ESC-2, J17 to PDB, J15 to RPI, J16 to Receiver, J12 to Servo, J5 to Servo, J6 to Servo, J8 to Servo, J13 to Servo, J10 to Servo, J11 to Servo, J4 to Servo, J9 to Servo, J7 to Servo
Connections:
- C1 pad 2: GND-WiFi -> GND
- C2 pad 2: GND-WiFi -> GND
- FC-TOP1 pad 83: Net-(FC-TOP1-GND-Pad83) -> GND
- NAV Module pad 2: Net-(FC-TOP1-GND-Pad83) -> GND
- NAV Module pad A2: Net-(FC-TOP1-GND-Pad83) -> GND
Routing:
- net GND: track 6.25 -> 26.4 mm
- net Net-(WiFi_module1-RST): track 26.8 -> 33.3 mm

Commit message: Reworked the WiFi module reset signal trace
Routing:
- net Net-(WiFi_module1-RST): vias 0 -> 1
